File: Hardware/imu.kicad_sch (KiCad schematic)
At the start: 9 parts, among them U3 MPU-6500, U4 MS5611-01BA

Commit message: nc
Parts:
- renumbered C2 to C15, C2 to C17, C2 to C18, R8 to R10, R6 to R11, R7 to R12
