File: Hardware/motor_controller.kicad_sch (KiCad schematic)
At the start: 16 parts, among them M1 53047-0210, M2 53047-0210, M3 53047-0210, M4 53047-0210, Q1 SIS434DN, Q2 SIS434DN, Q3 SIS434DN, Q4 SIS434DN

Commit message: nc
Parts:
- renumbered D1 to D4, D2 to D5, D3 to D6, D4 to D7, Q1 to Q4, Q2 to Q5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
