File: Hardware/power_management.kicad_sch (KiCad schematic)
At the start: 16 parts, among them J1 1S Lipo, J2 +, J3 -, Q1 IRLML6402, U1 TPS63031DSK

Commit message: nc
Parts:
- renumbered C2 to C1, C2 to C4, C2 to C5, C2 to C6, R1 to R2, R8 to R3
