File: Hardware/warnings.kicad_sch (KiCad schematic)
At the start: 11 parts, among them J5 LIGHT, Q2 MMBT3904, Q3 BC817, U6 5020

Commit message: nc
Parts:
- renumbered D6 to D2, D7 to D3, R17 to R13, R18 to R14, R17 to R15, R8 to R16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
